Commit message: Add pen link

File: drawbot/urdf/drawbot_tool.xacro (robot description, xacro)
@@ -1,18 +1,18 @@
 <?xml version="1.0" encoding="utf-8"?>
 <robot xmlns:xacro="https://ros.org/wiki/xacro">
-  <!-- Here we define the 2 parameters of the macro -->
   <xacro:macro name="drawbot_tool" params="prefix connected_to">
-    <!-- Create a fixed joint with a parameterized name. -->
     <joint name="${prefix}drawbot_joint" type="fixed">
-      <!-- The parent link must be read from the robot model it is attached to. -->
       <parent link="${connected_to}"/>
       <child link="${prefix}drawbot_tool"/>
-      <!-- The tool is directly attached to the flange. -->
       <origin rpy="3.14 3.14 0" xyz="0 0 -0.02"/>
+    </joint>
+    <joint name="${prefix}drawbot_pen_joint" type="fixed">
+      <parent link="${prefix}drawbot_tool"/>
+      <child link="${prefix}drawbot_tool_pen"/>
+      <origin rpy="0 0 0" xyz="0 -0.0475 0.0575"/>
     </joint>
     <link name="${prefix}drawbot_tool">
       <visual>
         <geometry>
-          <!-- The path to the visual meshes in the package. -->
           <mesh filename="package://drawbot/meshes/visual/tool.stl"/>
         </geometry>
@@ -20,6 +20,22 @@
       <collision>
         <geometry>
-          <!-- The path to the collision meshes in the package. -->
           <mesh filename="package://drawbot/meshes/collision/tool.stl"/>
+        </geometry>
+      </collision>
+    </link>
+    <link name="${prefix}drawbot_tool_pen">
+      <visual>
+        <origin xyz="0 0 0" rpy="0 0 0"/>
+        <geometry>
+          <cylinder radius="0.006" length="0.095"/>
+        </geometry>
+        <material name="Cyan">
+          <color rgba="0 1.0 1.0 1.0"/>
+        </material>
+      </visual>
+      <collision>
+        <origin xyz="0 0 0" rpy="0 0 0"/>
+        <geometry>
+          <cylinder radius="0.006" length="0.095"/>
         </geometry>
       </collision>

Commit message: Add moveit config

File: drawbot/urdf/drawbot_tool.xacro (robot description, xacro)
@@ -10,5 +10,10 @@
       <parent link="${prefix}drawbot_tool"/>
       <child link="${prefix}drawbot_tool_pen"/>
-      <origin rpy="0 0 0" xyz="0 -0.0475 0.0575"/>
+      <origin rpy="0 0 0" xyz="0 -0.0475 0.055"/>
+    </joint>
+    <joint name="${prefix}drawbot_pen_tip_joint" type="fixed">
+      <parent link="${prefix}drawbot_tool_pen"/>
+      <child link="${prefix}drawbot_tool_pen_tip"/>
+      <origin rpy="0 0 0" xyz="0 0 0.0475"/>
     </joint>
     <link name="${prefix}drawbot_tool">
@@ -28,5 +33,5 @@
         <origin xyz="0 0 0" rpy="0 0 0"/>
         <geometry>
-          <cylinder radius="0.006" length="0.095"/>
+          <cylinder radius="0.006" length="0.09"/>
         </geometry>
         <material name="Cyan">
@@ -37,5 +42,22 @@
         <origin xyz="0 0 0" rpy="0 0 0"/>
         <geometry>
-          <cylinder radius="0.006" length="0.095"/>
+          <cylinder radius="0.006" length="0.09"/>
+        </geometry>
+      </collision>
+    </link>
+    <link name="${prefix}drawbot_tool_pen_tip">
+      <visual>
+        <origin xyz="0 0 0" rpy="0 0 0"/>
+        <geometry>
+          <cylinder radius="0.003" length="0.005"/>
+        </geometry>
+        <material name="Green">
+          <color rgba="0 1.0 0 1.0"/>
+        </material>
+      </visual>
+      <collision>
+        <origin xyz="0 0 0" rpy="0 0 0"/>
+        <geometry>
+          <cylinder radius="0.003" length="0.005"/>
         </geometry>
       </collision>

Commit message: Draw board frame added

File: drawbot/urdf/drawbot_tool.xacro (robot description, xacro)
@@ -17,4 +17,13 @@
       <origin rpy="0 0 0" xyz="0 0 0.0475"/>
     </joint>
+    <!-- Define the draw board fixed frame with respect to the robot base -->
+    <joint name="${prefix}draw_board_fixed_joint" type="fixed">
+      <parent link="${prefix}base_link"/>
+      <child link="${prefix}draw_board"/>
+      <origin rpy="3.14 0 1.57" xyz="-0.554 0.308 0.025"/>
+    </joint>
+    <link name="${prefix}draw_board">
+      <origin xyz="-0.554 0.308 0.025"/>
+    </link>
     <link name="${prefix}drawbot_tool">
       <visual>

Commit message: Tool pen tip frame rotated to match draw board

File: drawbot/urdf/drawbot_tool.xacro (robot description, xacro)
@@ -15,5 +15,5 @@
       <parent link="${prefix}drawbot_tool_pen"/>
       <child link="${prefix}drawbot_tool_pen_tip"/>
-      <origin rpy="0 0 0" xyz="0 0 0.0475"/>
+      <origin rpy="0 0 3.14" xyz="0 0 0.0475"/>
     </joint>
     <!-- Define the draw board fixed frame with respect to the robot base -->

Commit message: working! first run

File: drawbot/urdf/drawbot_tool.xacro (robot description, xacro)
@@ -21,8 +21,8 @@
       <parent link="${prefix}base_link"/>
       <child link="${prefix}draw_board"/>
-      <origin rpy="3.14 0 1.57" xyz="-0.554 0.308 0.025"/>
+      <origin rpy="3.14 0 0.785" xyz="-0.554 0.308 0.0095"/>
     </joint>
     <link name="${prefix}draw_board">
-      <origin xyz="-0.554 0.308 0.025"/>
+      <origin xyz="-0.554 0.308 0.0095"/>
     </link>
     <link name="${prefix}drawbot_tool">
